File: AKBDB.kicad_sch (KiCad schematic)
At the start: 9 parts, among them J1 TYPE-C-31-M12_13, J2 SM04B-SRSS-TB(LF)(SN), U1 USBLC6-2SC6

Commit message: small fixes
Parts:
- R1, R2: footprint Resistor_SMD:R_0603_1608Metric -> Resistor_SMD:R_0402_1005Metric
Other:
- note added: "ESD + Fuse"
- note added: "JST"
- note removed: "ESD"
- note removed: "Misc"
- company: Designed by the keyboard community -> (none)
- title: Unified Daughterboard -> AKB DB
Changed lines of the file:
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@@
   (paper "A4")
   (title_block
-    (title "Unified Daughterboard")
+    (title "AKB DB")
     (date "2020-03-22")
-    (rev "C3")
-    (company "Designed by the keyboard community")
+    (rev "R1")
   )
   (junction (at 53.34 57.15) (diameter 0) (color 0 0 0 0)
@@
     (effects (font (size 5.08 5.08) (thickness 1.016) bold) (justify right bottom))
   )
-  (text "ESD" (at 117.475 138.43 180)
+  (text "ESD + Fuse" (at 134.62 137.16 180)
     (effects (font (size 5.08 5.08) (thickness 1.016) bold) (justify right bottom))
   )
-  (text "Misc" (at 257.81 137.16 180)
+  (text "JST" (at 257.81 137.16 180)
     (effects (font (size 5.08 5.08) (thickness 1.016) bold) (justify right bottom))
   )
@@
       (effects (font (size 0.762 0.762)))
     )
-    (property "Footprint" "Resistor_SMD:R_0603_1608Metric" (id 2) (at 57.15 48.26 0)
+    (property "Footprint" "Resistor_SMD:R_0402_1005Metric" (id 2) (at 57.15 48.26 0)
       (effects (font (size 1.27 1.27)) hide)
     )
@@
       (effects (font (size 0.762 0.762)))
     )
-    (property "Footprint" "Resistor_SMD:R_0603_1608Metric" (id 2) (at 57.15 50.8 0)
+    (property "Footprint" "Resistor_SMD:R_0402_1005Metric" (id 2) (at 57.15 50.8 0)
       (effects (font (size 1.27 1.27)) hide)
     )
@@
     )
     (path "/00000000-0000-0000-0000-00005c91b042"
-      (reference "R1") (unit 1) (value "5.1k") (footprint "Resistor_SMD:R_0603_1608Metric")
+      (reference "R1") (unit 1) (value "5.1k") (footprint "Resistor_SMD:R_0402_1005Metric")
     )
     (path "/00000000-0000-0000-0000-00005c91b0d9"
-      (reference "R2") (unit 1) (value "5.1k") (footprint "Resistor_SMD:R_0603_1608Metric")
+      (reference "R2") (unit 1) (value "5.1k") (footprint "Resistor_SMD:R_0402_1005Metric")
     )
     (path "/ab4d3cc6-46c6-4604-bd23-c61d13cacd62"
